Commit message: Generated map using slam_toolbox

File: ros2_RobotSimulation/factory_project/factory_amr_description/urdf/factory_amr1.xacro (robot description, xacro)
@@ -28,4 +28,11 @@
     <material>Gazebo/White</material>
   </gazebo>
+  <joint name="base_footprint_joint" type="fixed">
+        <parent link="base_link"/>
+        <child link="base_footprint"/>
+        <origin xyz="0 0 0" rpy="0 0 0"/>
+    </joint>
+    <link name="base_footprint">
+    </link>
   <link name="right_wheel_link">
     <inertial>

File: ros2_RobotSimulation/factory_project/factory_amr_description/urdf/factory_amr2.xacro (robot description, xacro)
@@ -28,4 +28,11 @@
     <material>Gazebo/White</material>
   </gazebo>
+  <joint name="base_footprint_joint" type="fixed">
+        <parent link="base_link"/>
+        <child link="base_footprint"/>
+        <origin xyz="0 0 0" rpy="0 0 0"/>
+    </joint>
+    <link name="base_footprint">
+    </link>
   <link name="right_wheel_link">
     <inertial>

File: ros2_RobotSimulation/factory_project/factory_amr_description/urdf/robot_urdf_1.xacro (robot description, xacro)
@@ -2,5 +2,5 @@
 <robot name="factory_amr1" xmlns:xacro="http://www.ros.org/wiki/xacro">
     <xacro:arg name="robot_namespace" default="factory_amr1"/>
-    <xacro:include filename="factory_amr.xacro"/>
+    <xacro:include filename="factory_amr1.xacro"/>
     <xacro:include filename="gazebo_control1.xacro"/>
     <!-- <xacro:include filename="lidar.xacro"/> -->

File: ros2_RobotSimulation/factory_project/factory_amr_description/urdf/robot_urdf_2.xacro (robot description, xacro)
@@ -2,5 +2,5 @@
 <robot name="factory_amr2" xmlns:xacro="http://www.ros.org/wiki/xacro">
     <xacro:arg name="robot_namespace" default="factory_amr2"/>
-    <xacro:include filename="factory_amr.xacro"/>
+    <xacro:include filename="factory_amr2.xacro"/>
     <xacro:include filename="gazebo_control2.xacro"/>
     <!-- <xacro:include filename="lidar.xacro"/> -->

File: ros2_RobotSimulation/factory_project/factory_amr_description/urdf/robot_urdf_3.xacro (robot description, xacro)
@@ -2,5 +2,5 @@
 <robot name="factory_amr3" xmlns:xacro="http://www.ros.org/wiki/xacro">
     <xacro:arg name="robot_namespace" default="factory_amr3"/>
-    <xacro:include filename="factory_amr.xacro"/>
+    <xacro:include filename="factory_amr3.xacro"/>
     <xacro:include filename="gazebo_control3.xacro"/>
     <!-- <xacro:include filename="lidar.xacro"/> -->

Commit message: navigation implementation completed

File: ros2_RobotSimulation/factory_project/factory_amr_description/urdf/factory_amr1.xacro (robot description, xacro)
@@ -8,5 +8,5 @@
     <inertial>
       <origin xyz="-0.002396599951463409 2.104073385822183e-15 0.2688636212913025" rpy="0 0 0"/>
-      <mass value="5"/>
+      <mass value="2"/>
       <inertia ixx="2.322166" iyy="2.720165" izz="3.470128" ixy="0.0" iyz="0.0" ixz="-0.006447"/>
     </inertial>
@@ -186,4 +186,5 @@
     <child link="right_wheel_link"/>
     <axis xyz="0.0 0.0 -1.0"/>
+    <limit effort="10" velocity="1.0"/>
   </joint>
   <joint name="left_wheel_joint" type="continuous">
@@ -192,4 +193,5 @@
     <child link="left_wheel_link"/>
     <axis xyz="0.0 0.0 1.0"/>
+    <limit effort="10" velocity="1.0"/>
   </joint>
   <joint name="luggage_joint" type="revolute">

File: ros2_RobotSimulation/factory_project/factory_amr_description/urdf/factory_amr2.xacro (robot description, xacro)
@@ -8,5 +8,5 @@
     <inertial>
       <origin xyz="-0.002396599951463409 2.104073385822183e-15 0.2688636212913025" rpy="0 0 0"/>
-      <mass value="5"/>
+      <mass value="2"/>
       <inertia ixx="2.322166" iyy="2.720165" izz="3.470128" ixy="0.0" iyz="0.0" ixz="-0.006447"/>
     </inertial>
@@ -186,4 +186,5 @@
     <child link="right_wheel_link"/>
     <axis xyz="0.0 0.0 -1.0"/>
+    <limit effort="10" velocity="1.0"/>
   </joint>
   <joint name="left_wheel_joint" type="continuous">
@@ -192,4 +193,5 @@
     <child link="left_wheel_link"/>
     <axis xyz="0.0 0.0 1.0"/>
+    <limit effort="10" velocity="1.0"/>
   </joint>
   <joint name="luggage_joint" type="revolute">

File: ros2_RobotSimulation/factory_project/factory_amr_description/urdf/factory_amr3.xacro (robot description, xacro)
@@ -8,5 +8,5 @@
     <inertial>
       <origin xyz="-0.002396599951463409 2.104073385822183e-15 0.2688636212913025" rpy="0 0 0"/>
-      <mass value="5"/>
+      <mass value="2"/>
       <inertia ixx="2.322166" iyy="2.720165" izz="3.470128" ixy="0.0" iyz="0.0" ixz="-0.006447"/>
     </inertial>
@@ -186,4 +186,5 @@
     <child link="right_wheel_link"/>
     <axis xyz="0.0 0.0 -1.0"/>
+    <limit effort="10" velocity="1.0"/>
   </joint>
   <joint name="left_wheel_joint" type="continuous">
@@ -192,4 +193,5 @@
     <child link="left_wheel_link"/>
     <axis xyz="0.0 0.0 1.0"/>
+    <limit effort="10" velocity="1.0"/>
   </joint>
   <joint name="luggage_joint" type="revolute">
@@ -255,5 +257,5 @@
               </ros>
               <output_type>sensor_msgs/LaserScan</output_type>
-              <frame_name>factory_amr2/laser_frame</frame_name>
+              <frame_name>factory_amr3/laser_frame</frame_name>
           </plugin>
       </sensor>
