Commit message: namespace added

File: ros2_RobotSimulation/factory_project/factory_amr_description/urdf/factory_amr.xacro (robot description, xacro)
@@ -120,24 +120,4 @@
     <material>Gazebo/Red</material>
   </gazebo>
-  <link name="camera_link">
-    <inertial>
-      <origin xyz="0.010000000000000064 0.0 0.0" rpy="0 0 0"/>
-      <mass value="0.19729201864543888"/>
-      <inertia ixx="3.9e-05" iyy="2.6e-05" izz="2.6e-05" ixy="0.0" iyz="-0.0" ixz="0.0"/>
-    </inertial>
-    <visual>
-      <origin xyz="-0.39 -0.0 -0.475" rpy="0 0 0"/>
-      <geometry>
-        <mesh filename="file://$(find factory_amr_description)/meshes/camera_1.stl" scale="0.001 0.001 0.001"/>
-      </geometry>
-      <material name="red"/>
-    </visual>
-    <collision>
-      <origin xyz="-0.39 -0.0 -0.475" rpy="0 0 0"/>
-      <geometry>
-        <mesh filename="file://$(find factory_amr_description)/meshes/camera_1.stl" scale="0.001 0.001 0.001"/>
-      </geometry>
-    </collision>
-  </link>
   <!-- caster wheels -->
   <joint name="front_caster" type="fixed">
@@ -218,15 +198,4 @@
     <child link="imu_link"/>
   </joint>
-  <joint name="camera_joint" type="fixed">
-    <origin xyz="0.39 0.0 0.475" rpy="0 0 0"/>
-    <parent link="base_link"/>
-    <child link="camera_link"/>
-  </joint>
-  <joint name="camera_optical_joint" type="fixed">
-    <origin xyz="0.0 0.0 0.0" rpy="${-pi/2} 0 ${-pi/2}"/>
-    <parent link="camera_link"/>
-    <child link="camera_optical_link"/>
-  </joint>
-  <link name="camera_optical_link" type="fixed"></link>
   <joint name="laser_joint" type="fixed">
       <origin xyz="0.0 0.0 0.26" rpy="0 0 0"/>
@@ -283,28 +252,3 @@
       </sensor>
   </gazebo>
-  <gazebo reference="camera_link">
-    <material>Gazebo/Red</material>
-    <sensor name="camera" type="camera">
-      <pose> 0 0 0 0 0 0 </pose>
-      <visualize>true</visualize>
-      <update_rate>10</update_rate>
-      <camera>
-        <horizontal_fov>1.089</horizontal_fov>
-        <image>
-          <format>B8G8R8</format>
-          <width>640</width>
-          <height>480</height>
-        </image>
-        <clip>
-          <near>0.05</near>
-          <far>8.0</far>
-        </clip>
-      </camera>
-      <plugin name="camera_controller" filename="libgazebo_ros_camera.so">
-        <frame_name>camera_optical_link</frame_name>
-        <min_depth>0.1</min_depth>
-        <max_depth>100.0</max_depth>
-      </plugin>
-    </sensor>
-  </gazebo>
 </robot>

File: ros2_RobotSimulation/factory_project/factory_amr_description/urdf/gazebo_control.xacro (robot description, xacro)
@@ -3,4 +3,6 @@
     <gazebo>
         <plugin name="diff_drive" filename="libgazebo_ros_diff_drive.so">
+            <robotNamespace>/$(arg robot_namespace)</robotNamespace>
+            <robotParam>/$(arg robot_namespace)/robot_description</robotParam>
             <left_joint>left_wheel_joint</left_joint>
             <right_joint>right_wheel_joint</right_joint>

File: ros2_RobotSimulation/factory_project/factory_amr_description/urdf/robot_urdf.xacro (robot description, xacro)
@@ -1,4 +1,5 @@
 <?xml version="1.0" ?>
 <robot name="factory_amr" xmlns:xacro="http://www.ros.org/wiki/xacro">
+    <xacro:arg name="robot_namespace" default=""/>
     <xacro:include filename="factory_amr.xacro"/>
     <xacro:include filename="gazebo_control.xacro"/>

Commit message: modified amr_urdf, nav2 parameters

File: ros2_RobotSimulation/factory_project/factory_amr_description/urdf/factory_amr.xacro (robot description, xacro)
@@ -127,5 +127,4 @@
     <material>Gazebo/Red</material>
   </gazebo>
-  <!-- caster wheels -->
   <joint name="front_caster" type="fixed">
     <parent link="base_link"/>
@@ -136,14 +135,14 @@
     <visual>
       <geometry>
-        <sphere radius="0.05"/>
-      </geometry>
-      <material name="black"/>
-    </visual>
-    <collision>
-      <geometry>
-        <sphere radius="0.05"/>
-      </geometry>
-    </collision>
-    <xacro:inertial_sphere mass="0.1" radius="0.05">
+        <sphere radius="0.03"/> <!-- Reduced size from 0.05 -->
+      </geometry>
+      <material name="black"/>
+    </visual>
+    <collision>
+      <geometry>
+        <sphere radius="0.03"/> <!-- Reduced size from 0.05 -->
+      </geometry>
+    </collision>
+    <xacro:inertial_sphere mass="0.1" radius="0.03"> <!-- Adjusted mass and radius -->
       <origin xyz="0 0 0" rpy="0 0 0"/>
     </xacro:inertial_sphere>
@@ -162,14 +161,14 @@
     <visual>
       <geometry>
-        <sphere radius="0.05"/>
-      </geometry>
-      <material name="black"/>
-    </visual>
-    <collision>
-      <geometry>
-        <sphere radius="0.05"/>
-      </geometry>
-    </collision>
-    <xacro:inertial_sphere mass="0.1" radius="0.05">
+        <sphere radius="0.03"/> <!-- Reduced size from 0.05 -->
+      </geometry>
+      <material name="black"/>
+    </visual>
+    <collision>
+      <geometry>
+        <sphere radius="0.03"/> <!-- Reduced size from 0.05 -->
+      </geometry>
+    </collision>
+    <xacro:inertial_sphere mass="0.1" radius="0.03"> <!-- Adjusted mass and radius -->
       <origin xyz="0 0 0" rpy="0 0 0"/>
     </xacro:inertial_sphere>
@@ -180,5 +179,4 @@
     <mu2 value="0.001"/>
   </gazebo>
-  <!-- joints -->
   <joint name="right_wheel_joint" type="continuous">
     <origin xyz="0.0 -0.25 0.1" rpy="${pi/2} 0 0"/>

File: ros2_RobotSimulation/factory_project/factory_amr_description/urdf/factory_amr1.xacro (robot description, xacro)
@@ -3,10 +3,10 @@
   <xacro:include filename="inertial_macros.xacro"/>
   <xacro:include filename="$(find factory_amr_description)/urdf/materials.xacro" />
-  <xacro:include filename="$(find factory_amr_description)/urdf/factory_amr.trans" />
+  <xacro:include filename="$(find factory_amr_description)/urdf/factory_amr1.trans" />
   <xacro:include filename="$(find factory_amr_description)/urdf/factory_amr.gazebo" />
   <link name="base_link">
     <inertial>
       <origin xyz="-0.002396599951463409 2.104073385822183e-15 0.2688636212913025" rpy="0 0 0"/>
-      <mass value="2"/>
+      <mass value="5"/>
       <inertia ixx="2.322166" iyy="2.720165" izz="3.470128" ixy="0.0" iyz="0.0" ixz="-0.006447"/>
     </inertial>
@@ -29,10 +29,9 @@
   </gazebo>
   <joint name="base_footprint_joint" type="fixed">
-        <parent link="base_link"/>
-        <child link="base_footprint"/>
-        <origin xyz="0 0 0" rpy="0 0 0"/>
-    </joint>
-    <link name="base_footprint">
-    </link>
+    <parent link="base_link"/>
+    <child link="base_footprint"/>
+    <origin xyz="0 0 0" rpy="0 0 0"/>
+  </joint>
+  <link name="base_footprint"/>
   <link name="right_wheel_link">
     <inertial>
@@ -127,5 +126,4 @@
     <material>Gazebo/Red</material>
   </gazebo>
-  <!-- caster wheels -->
   <joint name="front_caster" type="fixed">
     <parent link="base_link"/>
@@ -136,14 +134,14 @@
     <visual>
       <geometry>
-        <sphere radius="0.05"/>
-      </geometry>
-      <material name="black"/>
-    </visual>
-    <collision>
-      <geometry>
-        <sphere radius="0.05"/>
-      </geometry>
-    </collision>
-    <xacro:inertial_sphere mass="0.1" radius="0.05">
+        <sphere radius="0.03"/> <!-- Reduced size from 0.05 -->
+      </geometry>
+      <material name="black"/>
+    </visual>
+    <collision>
+      <geometry>
+        <sphere radius="0.03"/> <!-- Reduced size from 0.05 -->
+      </geometry>
+    </collision>
+    <xacro:inertial_sphere mass="0.1" radius="0.03"> <!-- Adjusted mass and radius -->
       <origin xyz="0 0 0" rpy="0 0 0"/>
     </xacro:inertial_sphere>
@@ -162,14 +160,14 @@
     <visual>
       <geometry>
-        <sphere radius="0.05"/>
-      </geometry>
-      <material name="black"/>
-    </visual>
-    <collision>
-      <geometry>
-        <sphere radius="0.05"/>
-      </geometry>
-    </collision>
-    <xacro:inertial_sphere mass="0.1" radius="0.05">
+        <sphere radius="0.03"/> <!-- Reduced size from 0.05 -->
+      </geometry>
+      <material name="black"/>
+    </visual>
+    <collision>
+      <geometry>
+        <sphere radius="0.03"/> <!-- Reduced size from 0.05 -->
+      </geometry>
+    </collision>
+    <xacro:inertial_sphere mass="0.1" radius="0.03"> <!-- Adjusted mass and radius -->
       <origin xyz="0 0 0" rpy="0 0 0"/>
     </xacro:inertial_sphere>
@@ -180,5 +178,4 @@
     <mu2 value="0.001"/>
   </gazebo>
-  <!-- joints -->
   <joint name="right_wheel_joint" type="continuous">
     <origin xyz="0.0 -0.25 0.1" rpy="${pi/2} 0 0"/>

File: ros2_RobotSimulation/factory_project/factory_amr_description/urdf/factory_amr2.xacro (robot description, xacro)
@@ -3,10 +3,10 @@
   <xacro:include filename="inertial_macros.xacro"/>
   <xacro:include filename="$(find factory_amr_description)/urdf/materials.xacro" />
-  <xacro:include filename="$(find factory_amr_description)/urdf/factory_amr.trans" />
+  <xacro:include filename="$(find factory_amr_description)/urdf/factory_amr2.trans" />
   <xacro:include filename="$(find factory_amr_description)/urdf/factory_amr.gazebo" />
   <link name="base_link">
     <inertial>
       <origin xyz="-0.002396599951463409 2.104073385822183e-15 0.2688636212913025" rpy="0 0 0"/>
-      <mass value="2"/>
+      <mass value="5"/>
       <inertia ixx="2.322166" iyy="2.720165" izz="3.470128" ixy="0.0" iyz="0.0" ixz="-0.006447"/>
     </inertial>
@@ -29,10 +29,9 @@
   </gazebo>
   <joint name="base_footprint_joint" type="fixed">
-        <parent link="base_link"/>
-        <child link="base_footprint"/>
-        <origin xyz="0 0 0" rpy="0 0 0"/>
-    </joint>
-    <link name="base_footprint">
-    </link>
+    <parent link="base_link"/>
+    <child link="base_footprint"/>
+    <origin xyz="0 0 0" rpy="0 0 0"/>
+  </joint>
+  <link name="base_footprint"/>
   <link name="right_wheel_link">
     <inertial>
@@ -127,5 +126,4 @@
     <material>Gazebo/Red</material>
   </gazebo>
-  <!-- caster wheels -->
   <joint name="front_caster" type="fixed">
     <parent link="base_link"/>
@@ -136,14 +134,14 @@
     <visual>
       <geometry>
-        <sphere radius="0.05"/>
-      </geometry>
-      <material name="black"/>
-    </visual>
-    <collision>
-      <geometry>
-        <sphere radius="0.05"/>
-      </geometry>
-    </collision>
-    <xacro:inertial_sphere mass="0.1" radius="0.05">
+        <sphere radius="0.03"/> <!-- Reduced size from 0.05 -->
+      </geometry>
+      <material name="black"/>
+    </visual>
+    <collision>
+      <geometry>
+        <sphere radius="0.03"/> <!-- Reduced size from 0.05 -->
+      </geometry>
+    </collision>
+    <xacro:inertial_sphere mass="0.1" radius="0.03"> <!-- Adjusted mass and radius -->
       <origin xyz="0 0 0" rpy="0 0 0"/>
     </xacro:inertial_sphere>
@@ -162,14 +160,14 @@
     <visual>
       <geometry>
-        <sphere radius="0.05"/>
-      </geometry>
-      <material name="black"/>
-    </visual>
-    <collision>
-      <geometry>
-        <sphere radius="0.05"/>
-      </geometry>
-    </collision>
-    <xacro:inertial_sphere mass="0.1" radius="0.05">
+        <sphere radius="0.03"/> <!-- Reduced size from 0.05 -->
+      </geometry>
+      <material name="black"/>
+    </visual>
+    <collision>
+      <geometry>
+        <sphere radius="0.03"/> <!-- Reduced size from 0.05 -->
+      </geometry>
+    </collision>
+    <xacro:inertial_sphere mass="0.1" radius="0.03"> <!-- Adjusted mass and radius -->
       <origin xyz="0 0 0" rpy="0 0 0"/>
     </xacro:inertial_sphere>
@@ -180,5 +178,4 @@
     <mu2 value="0.001"/>
   </gazebo>
-  <!-- joints -->
   <joint name="right_wheel_joint" type="continuous">
     <origin xyz="0.0 -0.25 0.1" rpy="${pi/2} 0 0"/>

File: ros2_RobotSimulation/factory_project/factory_amr_description/urdf/factory_amr3.xacro (robot description, xacro)
@@ -3,10 +3,10 @@
   <xacro:include filename="inertial_macros.xacro"/>
   <xacro:include filename="$(find factory_amr_description)/urdf/materials.xacro" />
-  <xacro:include filename="$(find factory_amr_description)/urdf/factory_amr.trans" />
+  <xacro:include filename="$(find factory_amr_description)/urdf/factory_amr3.trans" />
   <xacro:include filename="$(find factory_amr_description)/urdf/factory_amr.gazebo" />
   <link name="base_link">
     <inertial>
       <origin xyz="-0.002396599951463409 2.104073385822183e-15 0.2688636212913025" rpy="0 0 0"/>
-      <mass value="2"/>
+      <mass value="5"/>
       <inertia ixx="2.322166" iyy="2.720165" izz="3.470128" ixy="0.0" iyz="0.0" ixz="-0.006447"/>
     </inertial>
@@ -29,10 +29,9 @@
   </gazebo>
   <joint name="base_footprint_joint" type="fixed">
-        <parent link="base_link"/>
-        <child link="base_footprint"/>
-        <origin xyz="0 0 0" rpy="0 0 0"/>
-    </joint>
-    <link name="base_footprint">
-    </link>
+    <parent link="base_link"/>
+    <child link="base_footprint"/>
+    <origin xyz="0 0 0" rpy="0 0 0"/>
+  </joint>
+  <link name="base_footprint"/>
   <link name="right_wheel_link">
     <inertial>
@@ -127,5 +126,4 @@
     <material>Gazebo/Red</material>
   </gazebo>
-  <!-- caster wheels -->
   <joint name="front_caster" type="fixed">
     <parent link="base_link"/>
@@ -136,14 +134,14 @@
     <visual>
       <geometry>
-        <sphere radius="0.05"/>
-      </geometry>
-      <material name="black"/>
-    </visual>
-    <collision>
-      <geometry>
-        <sphere radius="0.05"/>
-      </geometry>
-    </collision>
-    <xacro:inertial_sphere mass="0.1" radius="0.05">
+        <sphere radius="0.03"/> <!-- Reduced size from 0.05 -->
+      </geometry>
+      <material name="black"/>
+    </visual>
+    <collision>
+      <geometry>
+        <sphere radius="0.03"/> <!-- Reduced size from 0.05 -->
+      </geometry>
+    </collision>
+    <xacro:inertial_sphere mass="0.1" radius="0.03"> <!-- Adjusted mass and radius -->
       <origin xyz="0 0 0" rpy="0 0 0"/>
     </xacro:inertial_sphere>
@@ -162,14 +160,14 @@
     <visual>
       <geometry>
-        <sphere radius="0.05"/>
-      </geometry>
-      <material name="black"/>
-    </visual>
-    <collision>
-      <geometry>
-        <sphere radius="0.05"/>
-      </geometry>
-    </collision>
-    <xacro:inertial_sphere mass="0.1" radius="0.05">
+        <sphere radius="0.03"/> <!-- Reduced size from 0.05 -->
+      </geometry>
+      <material name="black"/>
+    </visual>
+    <collision>
+      <geometry>
+        <sphere radius="0.03"/> <!-- Reduced size from 0.05 -->
+      </geometry>
+    </collision>
+    <xacro:inertial_sphere mass="0.1" radius="0.03"> <!-- Adjusted mass and radius -->
       <origin xyz="0 0 0" rpy="0 0 0"/>
     </xacro:inertial_sphere>
@@ -180,5 +178,4 @@
     <mu2 value="0.001"/>
   </gazebo>
-  <!-- joints -->
   <joint name="right_wheel_joint" type="continuous">
     <origin xyz="0.0 -0.25 0.1" rpy="${pi/2} 0 0"/>

File: ros2_RobotSimulation/factory_project/factory_amr_description/urdf/robot_urdf.xacro (robot description, xacro)
@@ -4,4 +4,3 @@
     <xacro:include filename="factory_amr.xacro"/>
     <xacro:include filename="gazebo_control.xacro"/>
-    <!-- <xacro:include filename="lidar.xacro"/> -->
 </robot>

File: ros2_RobotSimulation/factory_project/factory_amr_description/urdf/robot_urdf_1.xacro (robot description, xacro)
@@ -4,4 +4,3 @@
     <xacro:include filename="factory_amr1.xacro"/>
     <xacro:include filename="gazebo_control1.xacro"/>
-    <!-- <xacro:include filename="lidar.xacro"/> -->
 </robot>

File: ros2_RobotSimulation/factory_project/factory_amr_description/urdf/robot_urdf_2.xacro (robot description, xacro)
@@ -4,4 +4,3 @@
     <xacro:include filename="factory_amr2.xacro"/>
     <xacro:include filename="gazebo_control2.xacro"/>
-    <!-- <xacro:include filename="lidar.xacro"/> -->
 </robot>

File: ros2_RobotSimulation/factory_project/factory_amr_description/urdf/robot_urdf_3.xacro (robot description, xacro)
@@ -4,4 +4,3 @@
     <xacro:include filename="factory_amr3.xacro"/>
     <xacro:include filename="gazebo_control3.xacro"/>
-    <!-- <xacro:include filename="lidar.xacro"/> -->
 </robot>
