Commit message: modified controller

File: ros2_RobotSimulation/factory_project/factory_amr_description/urdf/amr1_ros2_control.xacro (robot description, xacro)
@@ -5,24 +5,8 @@
             <plugin>gazebo_ros2_control/GazeboSystem</plugin>
         </hardware>
-        <joint name="left_wheel_joint">
-            <command_interface name="velocity">
-                <param name="min">-10</param>
-                <param name="max">10</param>
-            </command_interface>
-            <state_interface name="velocity"/>
-            <state_interface name="position"/>
-        </joint>
-        <joint name="right_wheel_joint">
-            <command_interface name="velocity">
-                <param name="min">-10</param>
-                <param name="max">10</param>
-            </command_interface>
-            <state_interface name="velocity"/>
-            <state_interface name="position"/>
-        </joint>
         <joint name="luggage_joint">
             <command_interface name="position">
-                <param name="min">-10</param>
-                <param name="max">10</param>
+                <param name="min">0</param>
+                <param name="max">1</param>
             </command_interface>
             <state_interface name="velocity"/>
@@ -34,4 +18,19 @@
             <parameters>$(find factory_amr_description)/config/controller_factory_amr1.yaml</parameters>
         </plugin>
+        <plugin name="diff_drive" filename="libgazebo_ros_diff_drive.so">
+            <robotNamespace>factory_amr1</robotNamespace>
+            <robotParam>factory_amr1/robot_description</robotParam>
+            <left_joint>left_wheel_joint</left_joint>
+            <right_joint>right_wheel_joint</right_joint>
+            <wheel_separation>0.62</wheel_separation>
+            <wheel_diameter>1.0</wheel_diameter>
+            <max_wheel_torque>300</max_wheel_torque>
+            <max_wheel_acceleration>30.0</max_wheel_acceleration>
+            <odometry_frame>factory_amr1/odom</odometry_frame>
+            <robot_base_frame>factory_amr1/base_link</robot_base_frame>
+            <publish_odom>true</publish_odom>
+            <publish_odom_tf>true</publish_odom_tf>
+            <publish_wheel_tf>true</publish_wheel_tf>
+        </plugin>
     </gazebo>
 </robot>

File: ros2_RobotSimulation/factory_project/factory_amr_description/urdf/amr2_ros2_control.xacro (robot description, xacro)
@@ -5,24 +5,8 @@
             <plugin>gazebo_ros2_control/GazeboSystem</plugin>
         </hardware>
-        <joint name="left_wheel_joint">
-            <command_interface name="velocity">
-                <param name="min">-10</param>
-                <param name="max">10</param>
-            </command_interface>
-            <state_interface name="velocity"/>
-            <state_interface name="position"/>
-        </joint>
-        <joint name="right_wheel_joint">
-            <command_interface name="velocity">
-                <param name="min">-10</param>
-                <param name="max">10</param>
-            </command_interface>
-            <state_interface name="velocity"/>
-            <state_interface name="position"/>
-        </joint>
         <joint name="luggage_joint">
             <command_interface name="position">
-                <param name="min">-10</param>
-                <param name="max">10</param>
+                <param name="min">0</param>
+                <param name="max">1</param>
             </command_interface>
             <state_interface name="velocity"/>
@@ -34,4 +18,19 @@
             <parameters>$(find factory_amr_description)/config/controller_factory_amr2.yaml</parameters>
         </plugin>
+        <plugin name="diff_drive" filename="libgazebo_ros_diff_drive.so">
+            <robotNamespace>factory_amr2</robotNamespace>
+            <robotParam>factory_amr2/robot_description</robotParam>
+            <left_joint>left_wheel_joint</left_joint>
+            <right_joint>right_wheel_joint</right_joint>
+            <wheel_separation>0.62</wheel_separation>
+            <wheel_diameter>1.0</wheel_diameter>
+            <max_wheel_torque>300</max_wheel_torque>
+            <max_wheel_acceleration>30.0</max_wheel_acceleration>
+            <odometry_frame>factory_amr2/odom</odometry_frame>
+            <robot_base_frame>factory_amr2/base_link</robot_base_frame>
+            <publish_odom>true</publish_odom>
+            <publish_odom_tf>true</publish_odom_tf>
+            <publish_wheel_tf>true</publish_wheel_tf>
+        </plugin>
     </gazebo>
 </robot>

File: ros2_RobotSimulation/factory_project/factory_amr_description/urdf/amr3_ros2_control.xacro (robot description, xacro)
@@ -5,24 +5,8 @@
             <plugin>gazebo_ros2_control/GazeboSystem</plugin>
         </hardware>
-        <joint name="left_wheel_joint">
-            <command_interface name="velocity">
-                <param name="min">-10</param>
-                <param name="max">10</param>
-            </command_interface>
-            <state_interface name="velocity"/>
-            <state_interface name="position"/>
-        </joint>
-        <joint name="right_wheel_joint">
-            <command_interface name="velocity">
-                <param name="min">-10</param>
-                <param name="max">10</param>
-            </command_interface>
-            <state_interface name="velocity"/>
-            <state_interface name="position"/>
-        </joint>
         <joint name="luggage_joint">
             <command_interface name="position">
-                <param name="min">-10</param>
-                <param name="max">10</param>
+                <param name="min">0</param>
+                <param name="max">1</param>
             </command_interface>
             <state_interface name="velocity"/>
@@ -34,4 +18,19 @@
             <parameters>$(find factory_amr_description)/config/controller_factory_amr3.yaml</parameters>
         </plugin>
+        <plugin name="diff_drive" filename="libgazebo_ros_diff_drive.so">
+            <robotNamespace>factory_amr3</robotNamespace>
+            <robotParam>factory_amr3/robot_description</robotParam>
+            <left_joint>left_wheel_joint</left_joint>
+            <right_joint>right_wheel_joint</right_joint>
+            <wheel_separation>0.62</wheel_separation>
+            <wheel_diameter>1.0</wheel_diameter>
+            <max_wheel_torque>300</max_wheel_torque>
+            <max_wheel_acceleration>30.0</max_wheel_acceleration>
+            <odometry_frame>factory_amr3/odom</odometry_frame>
+            <robot_base_frame>factory_amr3/base_link</robot_base_frame>
+            <publish_odom>true</publish_odom>
+            <publish_odom_tf>true</publish_odom_tf>
+            <publish_wheel_tf>true</publish_wheel_tf>
+        </plugin>
     </gazebo>
 </robot>

File: ros2_RobotSimulation/factory_project/factory_amr_description/urdf/amr_ros2_control.xacro (robot description, xacro)
@@ -5,20 +5,4 @@
             <plugin>gazebo_ros2_control/GazeboSystem</plugin>
         </hardware>
-        <joint name="left_wheel_joint">
-            <command_interface name="velocity">
-                <param name="min">-10</param>
-                <param name="max">10</param>
-            </command_interface>
-            <state_interface name="velocity"/>
-            <state_interface name="position"/>
-        </joint>
-        <joint name="right_wheel_joint">
-            <command_interface name="velocity">
-                <param name="min">-10</param>
-                <param name="max">10</param>
-            </command_interface>
-            <state_interface name="velocity"/>
-            <state_interface name="position"/>
-        </joint>
         <joint name="luggage_joint">
             <command_interface name="position">
@@ -34,4 +18,17 @@
             <parameters>$(find factory_amr_description)/config/controller_factory_amr.yaml</parameters>
         </plugin>
+        <plugin name="diff_drive" filename="libgazebo_ros_diff_drive.so">
+            <left_joint>left_wheel_joint</left_joint>
+            <right_joint>right_wheel_joint</right_joint>
+            <wheel_separation>0.62</wheel_separation>
+            <wheel_diameter>1.0</wheel_diameter>
+            <max_wheel_torque>300</max_wheel_torque>
+            <max_wheel_acceleration>30.0</max_wheel_acceleration>
+            <odometry_frame>odom</odometry_frame>
+            <robot_base_frame>base_link</robot_base_frame>
+            <publish_odom>true</publish_odom>
+            <publish_odom_tf>true</publish_odom_tf>
+            <publish_wheel_tf>true</publish_wheel_tf>
+        </plugin>
     </gazebo>
 </robot>
